Commit message: Updated xacro and urdf
Signed-off-by: Mihir Kulkarni <mihirk284@gmail.com>

File: submitted_models/cerberus_gagarin_sensor_config_1/modelOrig.urdf (robot description, URDF)
Before this commit: robot GAGARIN, 5 links, 4 joints
Links:
- removed link ${name}/base_link
- removed link ${name}/rotor_0
- removed link ${name}/rotor_1
- removed link ${name}/rotor_2
- removed link ${name}/rotor_3
- added link base_link, mass 2.316; collision box size=0.5 0.5 0.4; visual box size=0.02 0.025 0.025
- added link rotor_0, mass 0.005; visual mesh filename=package://cerberus_gagarin_sensor_config_1/meshes/propeller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 scale=0.06 0.06 0.06
- added link rotor_1, mass 0.005; visual mesh filename=package://cerberus_gagarin_sensor_config_1/meshes/propeller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 scale=0.06 0.06 0.06
- added link rotor_2, mass 0.005; visual mesh filename=package://cerberus_gagarin_sensor_config_1/meshes/propeller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 scale=0.06 0.06 0.06
- added link rotor_3, mass 0.005; visual mesh filename=package://cerberus_gagarin_sensor_config_1/meshes/propeller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 scale=0.06 0.06 0.06
Joints:
- joint rotor_0_joint: child ${name}/rotor_0 -> rotor_0; limit lower=-1e+16 upper=1e+16 effort=-1 velocity=-1 -> lower=-1e+16 upper=1e+16 effort=0 velocity=0; origin xyz=0.2263 -0.2263 0.038 rpy=0 -0 0 -> xyz=0.1 -0.1 -0.035 rpy=0 -0 0; parent ${name}/base_link -> base_link
- joint rotor_1_joint: child ${name}/rotor_1 -> rotor_1; limit lower=-1e+16 upper=1e+16 effort=-1 velocity=-1 -> lower=-1e+16 upper=1e+16 effort=0 velocity=0; origin xyz=-0.2263 0.2263 0.038 rpy=0 -0 0 -> xyz=-0.1 0.1 -0.035 rpy=0 -0 0; parent ${name}/base_link -> base_link
- joint rotor_2_joint: child ${name}/rotor_2 -> rotor_2; limit lower=-1e+16 upper=1e+16 effort=-1 velocity=-1 -> lower=-1e+16 upper=1e+16 effort=0 velocity=0; origin xyz=0.2263 0.2263 0.038 rpy=0 -0 0 -> xyz=0.1 0.1 -0.035 rpy=0 -0 0; parent ${name}/base_link -> base_link
- joint rotor_3_joint: child ${name}/rotor_3 -> rotor_3; limit lower=-1e+16 upper=1e+16 effort=-1 velocity=-1 -> lower=-1e+16 upper=1e+16 effort=0 velocity=0; origin xyz=-0.2263 -0.2263 0.038 rpy=0 -0 0 -> xyz=-0.1 -0.1 -0.035 rpy=0 -0 0; parent ${name}/base_link -> base_link

File: submitted_models/cerberus_gagarin_sensor_config_1/urdf/model.xacro (robot description, xacro)
@@ -4,172 +4,152 @@
   <xacro:property name="name" value="$(arg name)"/>
   <link name='${name}/base_link'>
-    <inertial>
+      <inertial>
+        <origin xyz='0 0 0' rpy='0 -0 0'/>
+        <mass value='2.316'/>
+        <inertia ixx='0.017' ixy='0' ixz='0' iyy='0.018' iyz='0' izz='0.028'/>
+      </inertial>
+      <collision name='base_link_inertia_collision'>
+        <origin xyz='0 0 -0.224935' rpy='0 -0 0'/>
+        <geometry>
+          <box size='0.5 0.5 0.4'/>
+        </geometry>
+      </collision>
+      <visual name='base_link_inertia_visual'>
+        <origin xyz='0 0 -0.224935' rpy='0 -0 0'/>
+        <geometry>
+          <mesh filename='package://cerberus_gagarin_sensor_config_1/meshes/gagarin.dae' scale='1 1 1'/>
+        </geometry>
+      </visual>
+      <visual name='left_flashlight_led'>
+        <origin xyz='0.17757 0.17757 -0.017556' rpy='0 -0 2.35619'/>
+        <geometry>
+          <mesh filename='package://cerberus_gagarin_sensor_config_1/meshes/cree_xhp70.dae' scale='1 1 1'/>
+        </geometry>
+      </visual>
+      <visual name='right_flashlight_led'>
+        <origin xyz='0.17757 -0.17757 -0.017556' rpy='0 -0 0.785398'/>
+        <geometry>
+          <mesh filename='package://cerberus_gagarin_sensor_config_1/meshes/cree_xhp70.dae' scale='1 1 1'/>
+        </geometry>
+      </visual>
+      <visual name='camera_visual'>
+        <origin xyz='0.22 0 0.03' rpy='0 -0 0'/>
+        <geometry>
+          <box size='0.02 0.025 0.025'/>
+        </geometry>
+      </visual>
+      <visual name='laser_visual'>
+        <origin xyz='0 0 -0.05' rpy='3.14159 -0 0'/>
+        <geometry>
+          <cylinder radius='0.04041' length='0.0735'/>
+        </geometry>
+      </visual>
+    </link>
+    <sensor name='imu_sensor' update_rate='200'>
+      <parent link='${name}/base_link'/>
       <origin xyz='0 0 0' rpy='0 -0 0'/>
-      <mass value='3.76'/>
-      <inertia ixx='0.017' ixy='0' ixz='0' iyy='0.018' iyz='0' izz='0.028'/>
-    </inertial>
-    <collision name='base_link_inertia_collision'>
+    </sensor>
+    <sensor name='magnetometer' update_rate='20'>
+      <parent link='${name}/base_link'/>
       <origin xyz='0 0 0' rpy='0 -0 0'/>
-      <geometry>
-        <box size='0.82 0.82 0.375'/>
-      </geometry>
-    </collision>
-    <visual name='base_link_inertia_visual'>
-      <origin xyz='0 0 0' rpy='0 -0 0'/>
-      <geometry>
-        <mesh filename='package://cerberus_gagarin_sensor_config_1/meshes/gagarin.dae' scale='1 1 1'/>
-      </geometry>
-    </visual>
-    <visual name='left_flashlight_led'>
-      <origin xyz='0.247592 0.24728 -0.017556' rpy='0 -0 2.35619'/>
-      <geometry>
-        <mesh filename='package://cerberus_gagarin_sensor_config_1/meshes/cree_xhp70.dae' scale='1 1 1'/>
-      </geometry>
-    </visual>
-    <visual name='right_flashlight_led'>
-      <origin xyz='0.247592 -0.24728 -0.017556' rpy='0 -0 0.785398'/>
-      <geometry>
-        <mesh filename='package://cerberus_gagarin_sensor_config_1/meshes/cree_xhp70.dae' scale='1 1 1'/>
-      </geometry>
-    </visual>
-    <visual name='camera_visual'>
-      <origin xyz='0.172 0 -0.023' rpy='0 0.174533 0'/>
-      <geometry>
-        <box size='0.02 0.025 0.025'/>
-      </geometry>
-    </visual>
-    <visual name='laser_visual'>
-      <origin xyz='0 0 0.05' rpy='0 -0 0'/>
-      <geometry>
-        <cylinder radius='0.03' length='0.1'/>
-      </geometry>
-    </visual>
-  </link>
-  <sensor name='imu_sensor' update_rate='200'>
-    <parent link='${name}/base_link'/>
-    <origin xyz='0 0 0' rpy='0 -0 0'/>
-  </sensor>
-  <sensor name='magnetometer' update_rate='20'>
-    <parent link='${name}/base_link'/>
-    <origin xyz='0 0 0' rpy='0 -0 0'/>
-  </sensor>
-  <sensor name='camera_front' update_rate='20'>
-    <parent link='${name}/base_link'/>
-    <origin xyz='0.172 0 -0.023' rpy='0 0.174533 0'/>
-    <camera>
-      <image width='1440' height='1080' format='R8G8B8' hfov='2.0944' near='0.02' far='100' />
-    </camera>
-  </sensor>
-  <sensor name='front_laser' update_rate='10'>
-    <parent link='${name}/base_link'/>
-    <origin xyz='0 0 0.05' rpy='0 -0 0'/>
-  </sensor>
-  <link name='${name}/rotor_0'>
-    <inertial>
-      <origin xyz='0 0 0' rpy='0 -0 0'/>
-      <mass value='0.005'/>
-      <inertia ixx='9.75e-07' ixy='0' ixz='0' iyy='8.13545e-05' iyz='0' izz='8.22545e-05'/>
-    </inertial>
-    <collision name='rotor_0_collision'>
-      <origin xyz='0 0 0' rpy='0 -0 0'/>
-      <geometry>
-        <cylinder radius='0.175' length='0.005'/>
-      </geometry>
-    </collision>
-    <visual name='rotor_0_visual'>
-      <origin xyz='0 0 0' rpy='0 -0 0'/>
-      <geometry>
-        <mesh filename='package://cerberus_gagarin_sensor_config_1/meshes/m100_propeller_ccw.dae' scale='0.175 0.175 0.175'/>
-      </geometry>
-    </visual>
-  </link>
-  <link name='${name}/rotor_1'>
-    <inertial>
-      <origin xyz='0 0 0' rpy='0 -0 0'/>
-      <mass value='0.005'/>
-      <inertia ixx='9.75e-07' ixy='0' ixz='0' iyy='8.13545e-05' iyz='0' izz='8.22545e-05'/>
-    </inertial>
-    <collision name='rotor_1_collision'>
-      <origin xyz='0 0 0' rpy='0 -0 0'/>
-      <geometry>
-        <cylinder radius='0.175' length='0.005'/>
-      </geometry>
-    </collision>
-    <visual name='rotor_1_visual'>
-      <origin xyz='0 0 0' rpy='0 -0 0'/>
-      <geometry>
-        <mesh filename='package://cerberus_gagarin_sensor_config_1/meshes/m100_propeller_ccw.dae' scale='0.175 0.175 0.175'/>
-      </geometry>
-    </visual>
-  </link>
-  <link name='${name}/rotor_2'>
-    <inertial>
-      <origin xyz='0 0 0' rpy='0 -0 0'/>
-      <mass value='0.005'/>
-      <inertia ixx='9.75e-07' ixy='0' ixz='0' iyy='8.13545e-05' iyz='0' izz='8.22545e-05'/>
-    </inertial>
-    <collision name='rotor_2_collision'>
-      <origin xyz='0 0 0' rpy='0 -0 0'/>
-      <geometry>
-        <cylinder radius='0.175' length='0.005'/>
-      </geometry>
-    </collision>
-    <visual name='rotor_2_visual'>
-      <origin xyz='0 0 0' rpy='0 -0 0'/>
-      <geometry>
-        <mesh filename='package://cerberus_gagarin_sensor_config_1/meshes/m100_propeller_cw.dae' scale='0.175 0.175 0.175'/>
-      </geometry>
-    </visual>
-  </link>
-  <link name='${name}/rotor_3'>
-    <inertial>
-      <origin xyz='0 0 0' rpy='0 -0 0'/>
-      <mass value='0.005'/>
-      <inertia ixx='9.75e-07' ixy='0' ixz='0' iyy='8.13545e-05' iyz='0' izz='8.22545e-05'/>
-    </inertial>
-    <collision name='rotor_3_collision'>
-      <origin xyz='0 0 0' rpy='0 -0 0'/>
-      <geometry>
-        <cylinder radius='0.175' length='0.005'/>
-      </geometry>
-    </collision>
-    <visual name='rotor_3_visual'>
-      <origin xyz='0 0 0' rpy='0 -0 0'/>
-      <geometry>
-        <mesh filename='package://cerberus_gagarin_sensor_config_1/meshes/m100_propeller_cw.dae' scale='0.175 0.175 0.175'/>
-      </geometry>
-    </visual>
-  </link>
-  <joint name='rotor_0_joint' type='revolute'>
-    <origin xyz='0.2263 -0.2263 0.038' rpy='0 -0 0'/>
-    <parent link='${name}/base_link'/>
-    <child link='${name}/rotor_0'/>
-    <dynamics damping='0' friction='0' />
-    <axis xyz='0 0 1'/>
-    <limit lower='-1e+16' upper='1e+16' effort='0' velocity='0'/>
-  </joint>
-  <joint name='rotor_1_joint' type='revolute'>
-    <origin xyz='-0.2263 0.2263 0.038' rpy='0 -0 0'/>
-    <parent link='${name}/base_link'/>
-    <child link='${name}/rotor_1'/>
-    <dynamics damping='0' friction='0' />
-    <axis xyz='0 0 1'/>
-    <limit lower='-1e+16' upper='1e+16' effort='0' velocity='0'/>
-  </joint>
-  <joint name='rotor_2_joint' type='revolute'>
-    <origin xyz='0.2263 0.2263 0.038' rpy='0 -0 0'/>
-    <parent link='${name}/base_link'/>
-    <child link='${name}/rotor_2'/>
-    <dynamics damping='0' friction='0' />
-    <axis xyz='0 0 1'/>
-    <limit lower='-1e+16' upper='1e+16' effort='0' velocity='0'/>
-  </joint>
-  <joint name='rotor_3_joint' type='revolute'>
-    <origin xyz='-0.2263 -0.2263 0.038' rpy='0 -0 0'/>
-    <parent link='${name}/base_link'/>
-    <child link='${name}/rotor_3'/>
-    <dynamics damping='0' friction='0' />
-    <axis xyz='0 0 1'/>
-    <limit lower='-1e+16' upper='1e+16' effort='0' velocity='0'/>
-  </joint>
+    </sensor>
+    <sensor name='camera_front' update_rate='20'>
+      <parent link='${name}/base_link'/>
+      <origin xyz='0.23 0 0.03' rpy='0 -0 0'/>
+      <camera>
+        <image width='1440' height='1080' format='R8G8B8' hfov='2.0944' near='0.02' far='100' />
+      </camera>
+    </sensor>
+    <sensor name='front_laser' update_rate='10'>
+      <parent link='${name}/base_link'/>
+      <origin xyz='0 0 -0.05' rpy='3.14159 -0 0'/>
+    </sensor>
+    <sensor name='picoflexx' update_rate='5'>
+      <parent link='${name}/base_link'/>
+      <origin xyz='0 0 0.04' rpy='3.14159 -1.57079 3.14159'/>
+    </sensor>
+    <link name='${name}/rotor_0'>
+      <inertial>
+        <origin xyz='0 0 0' rpy='0 -0 0'/>
+        <mass value='0.005'/>
+        <inertia ixx='9.75e-07' ixy='0' ixz='0' iyy='8.13545e-05' iyz='0' izz='8.22545e-05'/>
+      </inertial>
+      <visual name='rotor_0_visual'>
+        <origin xyz='0 0 0' rpy='0 -0 0'/>
+        <geometry>
+          <mesh filename='package://cerberus_gagarin_sensor_config_1/meshes/propeller_ccw.dae' scale='0.06 0.06 0.06'/>
+        </geometry>
+      </visual>
+    </link>
+    <link name='${name}/rotor_1'>
+      <inertial>
+        <origin xyz='0 0 0' rpy='0 -0 0'/>
+        <mass value='0.005'/>
+        <inertia ixx='9.75e-07' ixy='0' ixz='0' iyy='8.13545e-05' iyz='0' izz='8.22545e-05'/>
+      </inertial>
+      <visual name='rotor_1_visual'>
+        <origin xyz='0 0 0' rpy='0 -0 0'/>
+        <geometry>
+          <mesh filename='package://cerberus_gagarin_sensor_config_1/meshes/propeller_ccw.dae' scale='0.06 0.06 0.06'/>
+        </geometry>
+      </visual>
+    </link>
+    <link name='${name}/rotor_2'>
+      <inertial>
+        <origin xyz='0 0 0' rpy='0 -0 0'/>
+        <mass value='0.005'/>
+        <inertia ixx='9.75e-07' ixy='0' ixz='0' iyy='8.13545e-05' iyz='0' izz='8.22545e-05'/>
+      </inertial>
+      <visual name='rotor_2_visual'>
+        <origin xyz='0 0 0' rpy='0 -0 0'/>
+        <geometry>
+          <mesh filename='package://cerberus_gagarin_sensor_config_1/meshes/propeller_cw.dae' scale='0.06 0.06 0.06'/>
+        </geometry>
+      </visual>
+    </link>
+    <link name='${name}/rotor_3'>
+      <inertial>
+        <origin xyz='0 0 0' rpy='0 -0 0'/>
+        <mass value='0.005'/>
+        <inertia ixx='9.75e-07' ixy='0' ixz='0' iyy='8.13545e-05' iyz='0' izz='8.22545e-05'/>
+      </inertial>
+      <visual name='rotor_3_visual'>
+        <origin xyz='0 0 0' rpy='0 -0 0'/>
+        <geometry>
+          <mesh filename='package://cerberus_gagarin_sensor_config_1/meshes/propeller_cw.dae' scale='0.06 0.06 0.06'/>
+        </geometry>
+      </visual>
+    </link>
+    <joint name='rotor_0_joint' type='revolute'>
+      <origin xyz='0.1 -0.1 -0.035' rpy='0 -0 0'/>
+      <parent link='${name}/base_link'/>
+      <child link='${name}/rotor_0'/>
+      <dynamics damping='0' friction='0' />
+      <axis xyz='0 0 1'/>
+      <limit lower='-1e+16' upper='1e+16' effort='0' velocity='0'/>
+    </joint>
+    <joint name='rotor_1_joint' type='revolute'>
+      <origin xyz='-0.1 0.1 -0.035' rpy='0 -0 0'/>
+      <parent link='${name}/base_link'/>
+      <child link='${name}/rotor_1'/>
+      <dynamics damping='0' friction='0' />
+      <axis xyz='0 0 1'/>
+      <limit lower='-1e+16' upper='1e+16' effort='0' velocity='0'/>
+    </joint>
+    <joint name='rotor_2_joint' type='revolute'>
+      <origin xyz='0.1 0.1 -0.035' rpy='0 -0 0'/>
+      <parent link='${name}/base_link'/>
+      <child link='${name}/rotor_2'/>
+      <dynamics damping='0' friction='0' />
+      <axis xyz='0 0 1'/>
+      <limit lower='-1e+16' upper='1e+16' effort='0' velocity='0'/>
+    </joint>
+    <joint name='rotor_3_joint' type='revolute'>
+      <origin xyz='-0.1 -0.1 -0.035' rpy='0 -0 0'/>
+      <parent link='${name}/base_link'/>
+      <child link='${name}/rotor_3'/>
+      <dynamics damping='0' friction='0' />
+      <axis xyz='0 0 1'/>
+      <limit lower='-1e+16' upper='1e+16' effort='0' velocity='0'/>
+    </joint>
 </robot>
